File: hardware/wr841n/wr841n-pic.brd (EAGLE design)
At the start: 49.7 x 49.5 mm, 40 parts, among them IC1 PIC18F26K80, IC2 ISO1050, IC3 ADUM1251, IC4 ADUM1201, IC5 ADUM1201

Commit message: CAN-CAN WR841N PCB wip
Parts:
- moved C6 1.85 mm to (23.5, 40.8)
Routing:
- net +18V: track 9.12 -> 10.3 mm
- net N$10: track 15.4 -> 16.5 mm
- net GND: track 167.1 -> 166.1 mm
- added copper zone on layer 1, net GND
- added copper zone on layer 16, net GND
- added copper zone on layer 1, net GNDA
- added copper zone on layer 16, net GNDA
Other:
- board text added: "SLCAN WR841N v8.x"
